File: hw/schematic/eagle/main.sch (EAGLE design)
At the start: 29 parts, among them IC1 DS1307, IC4 74LS595D, U1 ATMEGA328P_PDIP, U2 HEX_CONVERTER, Y1 32.768khz, Y2 16Mhz

Commit message: Schematic, Gerbers used in production
Parts:
- removed C3: 0.1uF, SparkFun-Passives:CAP1206
- removed J1_BTN_BLUE, J2_BTN_RED, J3_SW_YELLOW: (no value), SparkFun-Connectors:M03X2SHROUD
- removed J5_DISPLAY: (no value), SparkFun-Connectors:M05X2SHD
- removed JP1: JUMPER-PAD-3-NOYES_SILK, SparkFun-Passives:JUMPER-PAD-3-NOYES_SILK
- added J1: (no value), SparkFun-Connectors:M03LOCK
- added J2_UI_BTN: (no value), SparkFun-Connectors:M05X2SHD
- added J3: (no value), SparkFun-Connectors:M16PTH
- added Q1: MOSFET-NCHANNELBSS123LT1G, SparkFun-DiscreteSemi:MOSFET-NCHANNELBSS123LT1G
- added R6: 10kOhm, SparkFun-Resistors:RESISTOR1206
- added R7: 6 Ohm, SparkFun-Resistors:RESISTOR1206
- BAT1: value (none) -> Reverse
Connections:
- removed net ARDU_A0: U1.PC0(ADC0)
- removed net ARDU_A3: U1.PC3(ADC3)
- removed net ARDU_D2: U1.PD2(INT0)
- removed net ARDU_D3: U1.PD3(INT1)
- removed net ARDU_D4: J4_VIN_SIGNAL.3, R4.1, U1.PD4(XCK/T0)
- removed net ARDU_D7: U1.PD7(AIN1)
- removed net ARDU_D9: U1.PB1(OC1A)
- removed net ARDU_RX0: U1.PD1(TXD)
- removed net DP_LED: J5_DISPLAY.8
- removed net LED_ONOFF: J3_SW_YELLOW.3
- new net 1WIRE: J4_VIN_SIGNAL.1, R4.1, U1.PD4(XCK/T0)
- new net ARDU_TXO: J1.2, J4_VIN_SIGNAL.5, U1.PD1(TXD)
- new net BAT_MON: R6.2, U1.PC3(ADC3)
- new net DP_LED_K: J3.16, R7.2
- new net N$8: Q1.D, R7.1
- new net UI_DP_LED: Q1.G, U1.PD7(AIN1)
- net 3.3V: no longer C3.1
- net 5V: now also J3.15, J3.2; no longer J5_DISPLAY.1, JP1.2, JP1.3
- net ARDU_RXI: now also J1.3, J4_VIN_SIGNAL.3
- net BAT: now also R6.1
- net DP_DB4: now also J3.11; no longer J5_DISPLAY.9
- net DP_DB5: now also J3.12; no longer J5_DISPLAY.2
- net DP_DB6: now also J3.13; no longer J5_DISPLAY.4
- net DP_DB7: now also J3.14; no longer J5_DISPLAY.6
- net DP_E: now also J3.6; no longer J5_DISPLAY.7
- net DP_RS: now also J3.4; no longer J5_DISPLAY.5
- net DP_V0: now also J3.3; no longer J5_DISPLAY.3
- net EN: now also J2_UI_BTN.9; no longer J3_SW_YELLOW.1
- net GND: now also BAT1.-, J1.1, J2_UI_BTN.2, J2_UI_BTN.4, J2_UI_BTN.6, J2_UI_BTN.8, J3.1, Q1.S; no longer BAT1.+, C3.2, J1_BTN_BLUE.2, J1_BTN_BLUE.4, J1_BTN_BLUE.5, J1_BTN_BLUE.6, J2_BTN_RED.2, J2_BTN_RED.4, J2_BTN_RED.5, J2_BTN_RED.6, J3_SW_YELLOW.2, J3_SW_YELLOW.4, J3_SW_YELLOW.5, J3_SW_YELLOW.6, J4_VIN_SIGNAL.1, J4_VIN_SIGNAL.5, J5_DISPLAY.10
- net LB: now also U1.PB1(OC1A)
- net N$1: now also BAT1.+; no longer BAT1.-
- net SPI_CS_SD: now also U1.PB0(ICP)
- net UI_BTN_BLUE: now also J2_UI_BTN.1, U1.PD2(INT0); no longer J1_BTN_BLUE.1
- net UI_BTN_RED: now also J2_UI_BTN.5, U1.PD3(INT1); no longer J2_BTN_RED.1
- net UI_LED_BLUE: now also J2_UI_BTN.3, U1.PC1(ADC1); no longer J1_BTN_BLUE.3
- net UI_LED_RED: now also J2_UI_BTN.7, U1.PC0(ADC0); no longer J2_BTN_RED.3
- net VIN: now also J2_UI_BTN.10; no longer JP1.1
Other:
- note added: "ARDU_A0"
- note added: "ARDU_A1"
- note added: "ARDU_A3"
- note added: "ARDU_D2"
- note added: "ARDU_D3"
- note added: "ARDU_D4"
- note added: "ARDU_D7"
- note added: "ARDU_D9"
- note added: "FTDI_Connector"
- note removed: "1Wire"
- note removed: "?????"
- moved on the sheet: BAT1, R4
